Commit message: Added a seprate launch file for all things together, added gazebo ros control for diff_drive and a obstacle world

File: description/robot_core.xacro (robot description, xacro)
@@ -41,4 +41,7 @@
         </xacro:inertial_box>
     </link>
+    <gazebo reference="chassis">
+        <material>Gazebo/White</material>
+    </gazebo>
     <joint name="left_wheel_joint" type="continuous">
         <origin xyz="0.0 0.175 0.0" rpy="-${pi/2} 0.0 0.0"/>
@@ -67,4 +70,7 @@
         </collision>
     </link>
+    <gazebo reference="left_wheel">
+        <material> Gazebo/Blue</material>
+    </gazebo>
     <joint name="right_wheel_joint" type="continuous">
         <origin xyz="0.0 -0.175 0.0" rpy="${pi/2} 0.0 0.0"/>
@@ -93,4 +99,7 @@
         </collision>
     </link>
+    <gazebo reference="right_wheel">
+        <material> Gazebo/Blue</material>
+    </gazebo>
     <!-- CASTER WHEEL LINK -->
     <joint name="caster_wheel_joint" type="fixed">
@@ -119,3 +128,8 @@
         </collision>
     </link>
+    <gazebo reference="caster_wheel">
+        <material> Gazebo/Black</material>
+        <mu1 value="0.001"/>
+        <mu2 value="0.001"/>
+    </gazebo>
 </robot>
